File: Micro/65c21.kicad_sch (KiCad schematic)
At the start: 26 parts, among them J11 Internal I2C, J4 DE9_Plug_MountingHoles, J5 DE9_Plug_MountingHoles, J6 Conn_01x18, U16 74HC32, U20 W65C21SxPL, U25 74HC157

Commit message: Hardware: fixed error in schematic with clock moved dotclock to out 2 (better for jitter) allowed the replacement of 82c54 CPU CLK with CLK 2 moved nmi switch to a more reasonable location
Parts:
- TP21: footprint (none) -> TestPoint:TestPoint_Pad_D2.5mm
Changed lines of the file:
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@@
       (effects (font (size 1.27 1.27)))
     )
-    (property "Footprint" "" (at 175.26 81.28 0)
+    (property "Footprint" "TestPoint:TestPoint_Pad_D2.5mm" (at 175.26 81.28 0)
       (effects (font (size 1.27 1.27)) hide)
     )
