File: Micro/IO.kicad_sch (KiCad schematic)
At the start: 28 parts, among them J12 Debug Bank Select, J7 Conn_01x10, J8 I/0, U10 74HC154, U11 74HC154, U12 74HC273, U16 74HC32, U19 74HC86, U21 74HC02, U22 74HC32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

Commit message: Hardware: fixed error in schematic with clock moved dotclock to out 2 (better for jitter) allowed the replacement of 82c54 CPU CLK with CLK 2 moved nmi switch to a more reasonable location
Other:
- sheet 82c54 ports: added CLK2; removed none
Changed lines of the file:
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@@
     (effects (font (size 1.27 1.27)) (justify left))
+  )
+  (hierarchical_label "CLK2" (shape input) (at 129.54 124.46 180) (fields_autoplaced)
+    (effects (font (size 1.27 1.27)) (justify right))
   )
   (hierarchical_label "~{IRQ_SERIAL}" (shape input) (at 163.83 140.97 0) (fields_autoplaced)
@@
       (effects (font (size 1.27 1.27)) (justify right))
     )
-    (instances
+    (pin "CLK2" input (at 129.54 124.46 180)
+      (effects (font (size 1.27 1.27)) (justify left))
+    )
+    (instances

Commit message: Fixed error in TIE LE signal (Logic was inverted, replaced or with nor)
Parts:
- added unit 2 of U21
Connections:
- net GND: now also U22.10, U22.9
- net ~{WE}: now also U21.6; no longer U22.10
- net at U23.11 (LE): now also U21.4; no longer U22.8
- net at U22.11: now also U21.5; no longer U22.9
- no-connect marks 0 -> 1
Other:
- moved on the sheet: U22C
