File: Micro/6502.kicad_sch (KiCad schematic)
At the start: 15 parts, among them U1 W65C02SxQ, U2 AT28HC256BF, U3 IS62C256AL

Commit message: Finallized board, added jumpers for debug, added reset to Ext connector other errors fixed
Parts:
- added JP25: External Rom, Jumper:SolderJumper-2_P1.3mm_Bridged2Bar_RoundedPad1.0x1.5mm, symbol Jumper:SolderJumper_2_Bridged
- added JP26: External Rom, Connector_PinHeader_2.54mm:PinHeader_1x02_P2.54mm_Vertical, symbol Jumper:Jumper_2_Open
- added JP27: BE isolate, Jumper:SolderJumper-2_P1.3mm_Bridged2Bar_RoundedPad1.0x1.5mm, symbol Jumper:SolderJumper_2_Bridged
- added TP1: RDY, TestPoint:TestPoint_Pad_D2.0mm, symbol Connector:TestPoint
Connections:
- net +5V: now also JP27.1 (A)
- net ~{EEPROMCS}: now also JP25.2 (B), JP26.2 (B); no longer U2.20 (~{CE})
- net at U1.34 (BE): now also JP27.2 (B)
- net at R3.2, U1.41 (RDY): now also TP1.1
- new net: JP25.1 (A), JP26.1 (A), U2.20 (~{CE})
- no-connect marks 3 -> 2
Other:
- moved on the sheet: C8, JP15, R1, R2, R3, U1, tp32, tp33, tp34
