File: Micro/Micro.kicad_sch (KiCad schematic)
At the start: 27 parts, among them J13 Debug Misc, J9 Conn_02x20_Counter_Clockwise, SW1 Reset, SW2 SW_Push_Dual, U50 STM1061N38WX6F

Commit message: Hardware: fixed error in schematic with clock moved dotclock to out 2 (better for jitter) allowed the replacement of 82c54 CPU CLK with CLK 2 moved nmi switch to a more reasonable location
Other:
- sheet IO ports: added CLK2; removed none
Changed lines of the file:
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@@
 (kicad_sch (version 20230121) (generator eeschema)
   (paper "A4")
+  (junction (at 135.89 80.01) (diameter 0) (color 0 0 0 0)
+  )
   (junction (at 82.55 156.21) (diameter 0) (color 0 0 0 0)
   )
@@
     (stroke (width 0) (type default))
   )
+  (wire (pts (xy 180.34 27.94) (xy 180.34 80.01))
+    (stroke (width 0) (type default))
+  )
   (wire (pts (xy 73.66 60.96) (xy 90.17 60.96))
     (stroke (width 0) (type default))
@@
     (stroke (width 0) (type default))
   )
+  (wire (pts (xy 180.34 80.01) (xy 135.89 80.01))
+    (stroke (width 0) (type default))
+  )
   (wire (pts (xy 118.11 19.05) (xy 135.89 19.05))
     (stroke (width 0) (type default))
@@
     (stroke (width 0) (type default))
   )
+  (wire (pts (xy 118.11 27.94) (xy 180.34 27.94))
+    (stroke (width 0) (type default))
+  )
   (wire (pts (xy 73.66 68.58) (xy 82.55 68.58))
     (stroke (width 0) (type default))
@@
     (stroke (width 0) (type default))
   )
-  (wire (pts (xy 135.89 119.38) (xy 135.89 66.04))
+  (wire (pts (xy 135.89 119.38) (xy 135.89 80.01))
     (stroke (width 0) (type default))
   )
@@
   )
   (wire (pts (xy 223.52 106.68) (xy 223.52 107.95))
+    (stroke (width 0) (type default))
+  )
+  (wire (pts (xy 135.89 80.01) (xy 135.89 66.04))
     (stroke (width 0) (type default))
   )
@@
       (effects (font (size 1.27 1.27)) (justify right))
     )
+    (pin "CLK2" input (at 118.11 27.94 0)
+      (effects (font (size 1.27 1.27)) (justify right))
+    )

Commit message: Finallized board, added jumpers for debug, added reset to Ext connector other errors fixed
Parts:
- removed TP1: TestPoint, TestPoint:TestPoint_Pad_D2.5mm, symbol Connector:TestPoint
- added J14: EEPROM A14, Connector_PinHeader_2.54mm:PinHeader_1x01_P2.54mm_Vertical, symbol Connector_Generic:Conn_01x01
Connections:
- net CPU+RAM+ROM/EEPROMA14: now also J14.1 (Pin_1)
- net ~{RST}: now also J9.29 (Pin_29)
Changed lines of the file:
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@@
 (kicad_sch (version 20230121) (generator eeschema)
   (paper "A4")
+  (junction (at 96.52 88.9) (diameter 0) (color 0 0 0 0)
+  )
   (junction (at 135.89 80.01) (diameter 0) (color 0 0 0 0)
   )
@@
     (property "Intersheetrefs" "${INTERSHEET_REFS}" (at 13.8877 176.53 0)
       (effects (font (size 1.27 1.27)) (justify right) hide)
+    )
+  )
+  (global_label "~{RST}" (shape input) (at 223.52 88.9 0) (fields_autoplaced)
+    (effects (font (size 1.27 1.27)) (justify left))
+    (property "Intersheetrefs" "${INTERSHEET_REFS}" (at 229.9523 88.9 0)
+      (effects (font (size 1.27 1.27)) (justify left) hide)
     )
   )
@@
         (path "/5388c84f-02a4-4503-bb12-5559371e0a41"
           (reference "#PWR0125") (unit 1)
+        )
+      )
+    )
+  )
+  (symbol (lib_id "Connector_Generic:Conn_01x01") (at 96.52 93.98 270) (unit 1)
+    (in_bom yes) (on_board yes) (dnp no)
+    (property "Reference" "J14" (at 95.25 96.52 90)
+      (effects (font (size 1.27 1.27)) (justify left))
+    )
+    (property "Value" "EEPROM A14" (at 96.52 99.06 90)
+      (effects (font (size 1.27 1.27)) (justify left))
+    )
+    (property "Footprint" "Connector_PinHeader_2.54mm:PinHeader_1x01_P2.54mm_Vertical" (at 96.52 93.98 0)
+      (effects (font (size 1.27 1.27)) hide)
+    )
+    (property "Datasheet" "~" (at 96.52 93.98 0)
+      (effects (font (size 1.27 1.27)) hide)
+    )
+    (pin "1")
+    (instances
+      (project "Micro"
+        (path "/5388c84f-02a4-4503-bb12-5559371e0a41"
+          (reference "J14") (unit 1)
         )
       )
@@
         )
       )
-    )
-  )
-  (symbol (lib_id "Connector:TestPoint") (at 223.52 88.9 270) (unit 1)
-    (in_bom yes) (on_board yes) (dnp no)
-    (property "Reference" "TP1" (at 232.41 87.63 90)
-      (effects (font (size 1.27 1.27)) (justify left))
-    )
-    (property "Value" "TestPoint" (at 232.41 90.17 90)
-      (effects (font (size 1.27 1.27)) (justify left))
-    )
-    (property "Footprint" "TestPoint:TestPoint_Pad_D2.5mm" (at 223.52 93.98 0)
-      (effects (font (size 1.27 1.27)) hide)
-    )
-    (property "Datasheet" "~" (at 223.52 93.98 0)
-      (effects (font (size 1.27 1.27)) hide)
-    )
-    (pin "1")
-    (instances
-      (project "Micro"
-        (path "/5388c84f-02a4-4503-bb12-5559371e0a41"
-          (reference "TP1") (unit 1)
-        )
-      )
