File: Micro/power.kicad_sch (KiCad schematic)
At the start: 10 parts, among them J10 694106301002, U13 OKI-78SR-5, U51 AP2127K-3.3

Commit message: weird. idk why it made me change it
Parts:
- U51: value AP2127K-3.3 -> v-3.3
Changed lines of the file:
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@@
       (effects (font (size 1.27 1.27)))
     )
-    (property "Value" "AP2127K-3.3" (at 58.42 76.2 0)
+    (property "Value" "v-3.3" (at 58.42 76.2 0)
       (effects (font (size 1.27 1.27)))
     )

Commit message: Finallized board, added jumpers for debug, added reset to Ext connector other errors fixed
Parts:
- added JP28: Jumper_2_Open, Connector_PinHeader_2.54mm:PinHeader_1x02_P2.54mm_Vertical, symbol Jumper:Jumper_2_Open
Connections:
- net at J10.1 (POWER): now also JP28.1 (A); no longer F1.1
- new net: F1.1, JP28.2 (B)
Other:
- moved on the sheet: J10
Changed lines of the file:
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@@
   (junction (at 95.25 27.94) (diameter 0) (color 0 0 0 0)
   )
-  (junction (at 34.29 58.42) (diameter 0) (color 0 0 0 0)
-  )
   (junction (at 83.82 27.94) (diameter 0) (color 0 0 0 0)
   )
@@
   (junction (at 35.56 90.17) (diameter 0) (color 0 0 0 0)
   )
-  (wire (pts (xy 30.48 58.42) (xy 34.29 58.42))
+  (junction (at 24.13 58.42) (diameter 0) (color 0 0 0 0)
+  )
+  (wire (pts (xy 20.32 58.42) (xy 24.13 58.42))
     (stroke (width 0) (type default))
   )
@@
     (stroke (width 0) (type default))
   )
-  (wire (pts (xy 34.29 27.94) (xy 30.48 27.94))
+  (wire (pts (xy 24.13 27.94) (xy 20.32 27.94))
     (stroke (width 0) (type default))
   )
@@
     (stroke (width 0) (type default))
   )
-  (wire (pts (xy 30.48 27.94) (xy 30.48 58.42))
+  (wire (pts (xy 20.32 27.94) (xy 20.32 58.42))
+    (stroke (width 0) (type default))
+  )
+  (wire (pts (xy 24.13 58.42) (xy 25.4 58.42))
     (stroke (width 0) (type default))
   )
   (netclass_flag "" (length 2.54) (shape round) (at 36.83 27.94 0) (fields_autoplaced)
     (effects (font (size 1.27 1.27)) (justify left bottom))
-    (property "Netclass" "POWER" (at 37.5285 25.4 0)
+    (property "Netclass" "Power2" (at 37.5285 25.4 0)
       (effects (font (size 1.27 1.27) italic) (justify left))
     )
   )
-  (netclass_flag "" (length 2.54) (shape round) (at 48.26 27.94 180) (fields_autoplaced)
+  (netclass_flag "" (length 2.54) (shape round) (at 26.67 27.94 0) (fields_autoplaced)
+    (effects (font (size 1.27 1.27)) (justify left bottom))
+    (property "Netclass" "Power2" (at 27.3685 25.4 0)
+      (effects (font (size 1.27 1.27) italic) (justify left))
+    )
+  )
+  (netclass_flag "" (length 2.54) (shape round) (at 46.99 27.94 180) (fields_autoplaced)
     (effects (font (size 1.27 1.27)) (justify right bottom))
-    (property "Netclass" "POWER" (at 48.9585 30.48 0)
+    (property "Netclass" "Power2" (at 47.6885 30.48 0)
       (effects (font (size 1.27 1.27) italic) (justify left))
     )
   )
-  (netclass_flag "" (length 2.54) (shape round) (at 59.69 27.94 180) (fields_autoplaced)
+  (netclass_flag "" (length 2.54) (shape round) (at 60.96 27.94 180) (fields_autoplaced)
     (effects (font (size 1.27 1.27)) (justify right bottom))
-    (property "Netclass" "POWER" (at 60.3885 30.48 0)
+    (property "Netclass" "Power2" (at 61.6585 30.48 0)
       (effects (font (size 1.27 1.27) italic) (justify left))
     )
@@
     )
   )
-  (symbol (lib_id "SamacSys_Parts:694106301002") (at 34.29 58.42 90) (unit 1)
+  (symbol (lib_id "SamacSys_Parts:694106301002") (at 24.13 58.42 90) (unit 1)
     (in_bom yes) (on_board yes) (dnp no)
-    (property "Reference" "J10" (at 25.4 46.99 90)
+    (property "Reference" "J10" (at 15.24 46.99 90)
       (effects (font (size 1.27 1.27)) (justify right))
     )
-    (property "Value" "694106301002" (at 13.97 49.53 90)
+    (property "Value" "694106301002" (at 3.81 49.53 90)
       (effects (font (size 1.27 1.27)) (justify right))
     )
-    (property "Footprint" "SamacSys_Parts:694106301002_1" (at 31.75 31.75 0)
-      (effects (font (size 1.27 1.27)) (justify left) hide)
-    )
-    (property "Datasheet" "https://datasheet.datasheetarchive.com/originals/distributors/Datasheets_SAMA/1c153bd2ba42bb51bda59ee4cd9765cd.pdf" (at 34.29 31.75 0)
-      (effects (font (size 1.27 1.27)) (justify left) hide)
-    )
-    (property "Description" "WURTH ELEKTRONIK - 694106301002 - CONNECTOR, POWER ENTRY, JACK, 3A, 20VDC" (at 36.83 31.75 0)
-      (effects (font (size 1.27 1.27)) (justify left) hide)
-    )
-    (property "Height" "" (at 39.37 31.75 0)
-      (effects (font (size 1.27 1.27)) (justify left) hide)
-    )
-    (property "Mouser Part Number" "710-694106301002" (at 41.91 31.75 0)
-      (effects (font (size 1.27 1.27)) (justify left) hide)
-    )
-    (property "Mouser Price/Stock" "https://www.mouser.co.uk/ProductDetail/Wurth-Elektronik/694106301002?qs=a9WhcLg8qCwOEkcI62k5mA%3D%3D" (at 44.45 31.75 0)
-      (effects (font (size 1.27 1.27)) (justify left) hide)
-    )
-    (property "Manufacturer_Name" "Wurth Elektronik" (at 46.99 31.75 0)
-      (effects (font (size 1.27 1.27)) (justify left) hide)
-    )
-    (property "Manufacturer_Part_Number" "694106301002" (at 49.53 31.75 0)
+    (property "Footprint" "SamacSys_Parts:694106301002_1" (at 21.59 31.75 0)
+      (effects (font (size 1.27 1.27)) (justify left) hide)
+    )
+    (property "Datasheet" "https://datasheet.datasheetarchive.com/originals/distributors/Datasheets_SAMA/1c153bd2ba42bb51bda59ee4cd9765cd.pdf" (at 24.13 31.75 0)
+      (effects (font (size 1.27 1.27)) (justify left) hide)
+    )
+    (property "Description" "WURTH ELEKTRONIK - 694106301002 - CONNECTOR, POWER ENTRY, JACK, 3A, 20VDC" (at 26.67 31.75 0)
+      (effects (font (size 1.27 1.27)) (justify left) hide)
+    )
+    (property "Height" "" (at 29.21 31.75 0)
+      (effects (font (size 1.27 1.27)) (justify left) hide)
+    )
+    (property "Mouser Part Number" "710-694106301002" (at 31.75 31.75 0)
+      (effects (font (size 1.27 1.27)) (justify left) hide)
+    )
+    (property "Mouser Price/Stock" "https://www.mouser.co.uk/ProductDetail/Wurth-Elektronik/694106301002?qs=a9WhcLg8qCwOEkcI62k5mA%3D%3D" (at 34.29 31.75 0)
+      (effects (font (size 1.27 1.27)) (justify left) hide)
+    )
+    (property "Manufacturer_Name" "Wurth Elektronik" (at 36.83 31.75 0)
+      (effects (font (size 1.27 1.27)) (justify left) hide)
+    )
+    (property "Manufacturer_Part_Number" "694106301002" (at 39.37 31.75 0)
       (effects (font (size 1.27 1.27)) (justify left) hide)
     )
@@
     )
   )
-  (symbol (lib_id "power:GND") (at 34.29 58.42 0) (unit 1)
-    (in_bom yes) (on_board yes) (dnp no) (fields_autoplaced)
-    (property "Reference" "#PWR0174" (at 34.29 64.77 0)
-      (effects (font (size 1.27 1.27)) hide)
-    )
-    (property "Value" "GND" (at 34.29 63.5 0)
-      (effects (font (size 1.27 1.27)))
-    )
-    (property "Footprint" "" (at 34.29 58.42 0)
-      (effects (font (size 1.27 1.27)) hide)
-    )
-    (property "Datasheet" "" (at 34.29 58.42 0)
+  (symbol (lib_id "power:GND") (at 25.4 58.42 0) (unit 1)
+    (in_bom yes) (on_board yes) (dnp no) (fields_autoplaced)
+    (property "Reference" "#PWR0174" (at 25.4 64.77 0)
+      (effects (font (size 1.27 1.27)) hide)
+    )
+    (property "Value" "GND" (at 25.4 63.5 0)
+      (effects (font (size 1.27 1.27)))
+    )
+    (property "Footprint" "" (at 25.4 58.42 0)
+      (effects (font (size 1.27 1.27)) hide)
+    )
+    (property "Datasheet" "" (at 25.4 58.42 0)
       (effects (font (size 1.27 1.27)) hide)
     )
@@
         )
       )
+    )
+  )
+  (symbol (lib_id "Jumper:Jumper_2_Open") (at 31.75 27.94 0) (unit 1)
+    (in_bom yes) (on_board yes) (dnp no)
+    (property "Reference" "JP28" (at 31.75 21.59 0)
+      (effects (font (size 1.27 1.27)))
+    )
+    (property "Value" "Jumper_2_Open" (at 27.94 24.13 0)
+      (effects (font (size 1.27 1.27)))
+    )
+    (property "Footprint" "Connector_PinHeader_2.54mm:PinHeader_1x02_P2.54mm_Vertical" (at 31.75 27.94 0)
+      (effects (font (size 1.27 1.27)) hide)
+    )
+    (property "Datasheet" "~" (at 31.75 27.94 0)
+      (effects (font (size 1.27 1.27)) hide)
+    )
+    (pin "1")
+    (pin "2")
+    (instances
+      (project "Micro"
+        (path "/5388c84f-02a4-4503-bb12-5559371e0a41/04286a1a-b9f0-4501-b37a-2901cf88a3e5"
+          (reference "JP28") (unit 1)
+        )
+      )
